File: _autosave-Project.kicad_sch (KiCad schematic)
At the start: 101 parts, among them IC1 CH224K, IC2 TPS27081ADDCR, IC3 TPS5430DDAR, IC4 TP4056-42-ESOP8, IC5 TPAP2112K-3.3TRG1, IC6 TPS27081ADDCR, J1 Conn_02x16_Odd_Even, J2 TYPE-C-31-M-12, J3 Conn_01x02, Q1 AO3400A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

Commit message: Add files via upload
Parts:
- L1: LCSC C167969C408452 -> C408452
Changed lines of the file:
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@@
       (effects (font (size 1.27 1.27)) hide)
     )
-    (property "LCSC" "C167969C408452" (at 130.175 41.91 90)
+    (property "LCSC" "C408452" (at 130.175 41.91 90)
       (effects (font (size 1.27 1.27)) hide)
     )
