File: Project-backups/Project.kicad_sch (KiCad schematic)
At the start: 101 parts, among them IC1 CH224K, IC2 TPS27081ADDCR, IC3 TPS5430DDAR, IC4 TP4056-42-ESOP8, IC5 TPAP2112K-3.3TRG1, IC6 TPS27081ADDCR, J1 Conn_02x16_Odd_Even, J2 TYPE-C-31-M-12, J3 Conn_01x02, Q1 AO3400A, U1 INA219AxDCN, U3 MT3608, U4 DRV8833PWP, U5 DRV8833PWP

Commit message: Add files via upload
Parts:
- removed FB1: FerriteBead, GZ1608D601TF:BEADC1608X95N, symbol Device:FerriteBead
- removed IC5: TPAP2112K-3.3TRG1, TPAP2112K-3.3TRG1:SOT95P280X125-5N, symbol TPAP2112K-3_3TRG1:TPAP2112K-3.3TRG1
- removed J3: Conn_01x02, Connector_JST:JST_PH_S2B-PH-K_1x02_P2.00mm_Horizontal, symbol Connector_Generic:Conn_01x02
- removed S1: SS-12D11G3R, SS-12D11G3R:SS12D11G3R, symbol SS-12D11G3R:SS-12D11G3R
- added U2: NCV8114ASN120T1G, Package_TO_SOT_SMD:TSOT-23-5, symbol Regulator_Linear:NCV8114ASN120T1G
- D1, D3: LCSC C8678 -> (none)
- IC1: LCSC C970725 -> (none)
- IC2, IC6: LCSC C128404 -> (none)
- IC3: LCSC C9864 -> (none)
- IC4: LCSC C16581 -> (none)
- J1: footprint Connector_PinHeader_2.54mm:PinHeader_2x16_P2.54mm_Vertical -> (none)
- JP1, JP2, JP3: footprint Jumper:SolderJumper-2_P1.3mm_Open_TrianglePad1.0x1.5mm -> (none)
- L1: value 15uH -> 15uH+; footprint Inductor_SMD:L_Sunlord_MWSA0603S -> (none); LCSC C167969C408452 -> (none)
- Q1: LCSC C20917 -> (none)
- R1: footprint Resistor_SMD:R_0603_1608Metric -> (none); LCSC C23204 -> (none)
- R10, R12, R15: footprint Resistor_SMD:R_0805_2012Metric -> (none); LCSC C17444 -> C22790
- R11: footprint Resistor_SMD:R_0805_2012Metric -> (none); LCSC C17560 -> C31850
- R13, R16, R2: footprint Resistor_SMD:R_0805_2012Metric -> (none); LCSC C17470 -> C22807
- R14, R17: footprint Resistor_SMD:R_0805_2012Metric -> (none); LCSC C17414 -> C25804
- R18, R19, R20, R21, R24, R25: value 1R -> 1; footprint Resistor_SMD:R_0603_1608Metric -> KiCad:RESC1608X55N
- R22, R23: value 2R -> 2; footprint Resistor_SMD:R_0603_1608Metric -> 2 OHM:RESC1608X55N
- R3: footprint Resistor_SMD:R_0805_2012Metric -> (none); LCSC C4382 -> (none)
- R4, R6: footprint Resistor_SMD:R_0603_1608Metric -> (none); LCSC C13167 -> (none)
- R5, R8: footprint Resistor_SMD:R_0805_2012Metric -> (none); LCSC C17414 -> (none)
- R7: footprint Resistor_SMD:R_1206_3216Metric -> (none); LCSC C4410 -> (none)
- TP1, TP10, TP11, TP12, TP13, TP14, TP15, TP16, TP17, TP18, TP19, TP2, TP20, TP21, TP22, TP23, TP24, TP25, TP26, TP27, TP28, TP29, TP3, TP4, TP5, TP6, TP7, TP8, TP9: footprint TestPoint:TestPoint_Pad_D1.5mm -> (none)
- U1: LCSC C87469 -> (none)
Connections:
- net ANAL_GND is gone; now on net GND: U1.3 (GND), U1.8 (A1)
- net Bat_out is gone; now on net Battery: R26.2, R27.2, R28.2, R9.2, TP5.1, U1.1 (IN+)
- net Charging is gone; now on net Battery: JP3.1 (A)
- net +5V: no longer C21.1
- net 3V3 Out: now also U2.5 (OUT)
- net 5V Out: no longer IC2.5 (ON/OFF), J1.25 (Pin_25), R14.1, TP13.1
- net Battery: now also C13.2, C15.1, C16.2, C18.1, C7.2, C9.2, U3.5 (IN), U4.12 (VM), U5.12 (VM), U2.1 (IN)
- net GND: now also U2.2 (GND)
- removed net Monitor_out: C13.2, C15.1, C16.2, C18.1, C7.2, C9.2, R26.1, R27.1, R28.1, R9.1, TP6.1, U1.2 (IN-), U3.4 (EN), U3.5 (IN), U4.1 (nSLEEP), U4.12 (VM), U5.1 (nSLEEP), U5.12 (VM)
- new net CTRL_EXT_LOAD1: IC2.5 (ON/OFF), J1.25 (Pin_25), R14.1, TP13.1
- new net Load: R26.1, R27.1, R28.1, R9.1, TP6.1, U1.2 (IN-)
- new net Switch Out: U2.3 (EN), U3.4 (EN), U4.1 (nSLEEP), U5.1 (nSLEEP)
Other:
- note added: "2x external load switches"
- note removed: "2x External Load Switches"
- note removed: "H-Bridge Drivers"
- note removed: "Not sure where switch is supposed to go"
- note removed: "~ an LED show that the battery is charging? I rate if there is enough in budget at the end, but otherwise dont bother"
- note removed: "~Found footprint/component for inductor (*IT IS EXTENDED THOUGH) datashit,part # and footprint are added to 15uH+"
- moved on the sheet: C10, C11, C12, C13, C14, C15, C16, C17, C18, C19, C20, C21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
